File: slu.kicad_pcb (KiCad board)
At the start: 2 copper layers, 99.6 x 100.9 mm, 168 parts, among them J1 lcd_out, sw1 sw_2pos

Commit message: started ico2 cleanup
Routing:
- net /ICD11: track 17.0 -> 13.7 mm
- net /ICD13: track 31.8 -> 34.7 mm, vias 5 -> 6
- net /ICD9: track 48.6 -> 46.0 mm
- net /SER1-2: track 96.9 -> 94.8 mm
- net /ICD16: track 30.4 -> 28.7 mm
- net /ICD63: track 106.8 -> 106.1 mm
- net /ICD10: track 33.5 -> 33.0 mm
- net /ICD15: track 25.2 -> 25.0 mm, vias 4 -> 6

Commit message: some finishing touches
Parts:
- moved r34 0.72 mm to (76.7, 142.0)
- moved r35 0.47 mm to (76.7, 139.6)
- moved r36 0.35 mm to (76.7, 137.2)
Routing:
- net /ICD26: track 31.8 -> 23.6 mm, vias 2 -> 4
- net /SER5-6: track 174.4 -> 166.6 mm
- net /ICD4: track 30.8 -> 23.0 mm
- net /OE: track 384.5 -> 391.1 mm, vias 35 -> 29
- net /ICD13: track 34.7 -> 29.8 mm, vias 6 -> 8
- net /SER6-7: track 84.4 -> 79.8 mm
- net /ICD58: track 59.4 -> 63.2 mm
- net /ICD14: track 27.3 -> 23.5 mm
- net /ICD16: track 28.7 -> 25.4 mm
- net /ICD23: track 30.2 -> 27.0 mm
- net +5V: track 281.3 -> 284.5 mm
- net /ICD41: track 40.3 -> 43.5 mm, vias 0 -> 2
- net Net-(a1-D13): track 115.9 -> 119.0 mm
- net /SCK(CP): track 89.3 -> 92.3 mm
- net /ICD9: track 46.0 -> 48.9 mm, vias 4 -> 6
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